File: CAN-FD Shield.brd (EAGLE design)
At the start: 68.8 x 53.5 mm, 38 parts, among them J2 JUMPER-3P-SHORT, J3 JUMPER-3P-SHORT, J4 JUMPER-3P-SHORT, J5 JUMPER-3P-SHORT, U5 MCP2517FD, U6 MCP2542, X2 20MHz

Commit message: update
Parts:
- moved U$5 28.8 mm to (-0.73, -7.49)
Changed lines of the file:
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@@
 <grid distance="5" unitdist="mil" unit="mil" style="lines" multiple="5" display="yes" altdistance="2.5" altunitdist="mil" altunit="mil"/>
 <layers>
-<layer number="1" name="Top" color="4" fill="1" visible="no" active="yes"/>
-<layer number="16" name="Bottom" color="1" fill="1" visible="no" active="yes"/>
-<layer number="17" name="Pads" color="2" fill="1" visible="no" active="yes"/>
-<layer number="18" name="Vias" color="2" fill="1" visible="no" active="yes"/>
-<layer number="19" name="Unrouted" color="6" fill="1" visible="no" active="yes"/>
+<layer number="1" name="Top" color="4" fill="1" visible="yes" active="yes"/>
+<layer number="16" name="Bottom" color="1" fill="1" visible="yes" active="yes"/>
+<layer number="17" name="Pads" color="2" fill="1" visible="yes" active="yes"/>
+<layer number="18" name="Vias" color="2" fill="1" visible="yes" active="yes"/>
+<layer number="19" name="Unrouted" color="6" fill="1" visible="yes" active="yes"/>
 <layer number="20" name="Dimension" color="5" fill="1" visible="yes" active="yes"/>
 <layer number="21" name="tPlace" color="7" fill="1" visible="yes" active="yes"/>
-<layer number="22" name="bPlace" color="3" fill="1" visible="no" active="yes"/>
-<layer number="23" name="tOrigins" color="15" fill="1" visible="no" active="yes"/>
-<layer number="24" name="bOrigins" color="3" fill="1" visible="no" active="yes"/>
-<layer number="25" name="tNames" color="7" fill="1" visible="no" active="yes"/>
-<layer number="26" name="bNames" color="3" fill="1" visible="no" active="yes"/>
-<layer number="27" name="tValues" color="7" fill="1" visible="yes" active="yes"/>
+<layer number="22" name="bPlace" color="3" fill="1" visible="yes" active="yes"/>
+<layer number="23" name="tOrigins" color="15" fill="1" visible="yes" active="yes"/>
+<layer number="24" name="bOrigins" color="3" fill="1" visible="yes" active="yes"/>
+<layer number="25" name="tNames" color="7" fill="1" visible="yes" active="yes"/>
+<layer number="26" name="bNames" color="3" fill="1" visible="yes" active="yes"/>
+<layer number="27" name="tValues" color="7" fill="1" visible="no" active="yes"/>
 <layer number="28" name="bValues" color="7" fill="1" visible="no" active="yes"/>
 <layer number="29" name="tStop" color="7" fill="3" visible="no" active="yes"/>
@@
 <layer number="43" name="vRestrict" color="2" fill="10" visible="no" active="yes"/>
 <layer number="44" name="Drills" color="7" fill="1" visible="no" active="yes"/>
-<layer number="45" name="Holes" color="7" fill="1" visible="yes" active="yes"/>
+<layer number="45" name="Holes" color="7" fill="1" visible="no" active="yes"/>
 <layer number="46" name="Milling" color="3" fill="1" visible="no" active="yes"/>
 <layer number="47" name="Measures" color="7" fill="1" visible="no" active="yes"/>
@@
 <attribute name="VALUE" x="37.084" y="34.544" size="0.889" layer="28" ratio="11" rot="MR180"/>
 </element>
-<element name="U$5" library="moudle-new" package="SEEEDSTUDIO-PCB-FRAME" value="SEEEDSTUDIO-OPEN-SCH-FRAME" x="18.700109375" y="-28.702" smashed="yes"/>
+<element name="U$5" library="moudle-new" package="SEEEDSTUDIO-PCB-FRAME" value="SEEEDSTUDIO-OPEN-SCH-FRAME" x="-0.730890625" y="-7.493" smashed="yes"/>
 <element name="J2" library="Discrete-new" package="3P-SMD-SHORT" value="JUMPER-3P-SHORT" x="19.05" y="34.544" smashed="yes" rot="MR180">
 <attribute name="NAME" x="18.415" y="34.544" size="0.3048" layer="34" ratio="10" rot="MR180"/>

Commit message: update
Parts:
- U$1: device Logo:LOGO_SILK -> Longan-LOGO:LONGAN-SILK-SMALLER
- moved U$1 13.4 mm to (45.2, 18.9)
Other:
- board text added: "by Longan Labs"
- board text added: "longan-labs.cc"
- board text removed: "by Seeed Studio"
- board text removed: "wiki.seeed.cc/can"
Changed lines of the file:
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@@
 <text x="43.942" y="18.161" size="1.27" layer="22" ratio="12" rot="MR0">CAN-FD Shield</text>
 <text x="43.942" y="15.621" size="1.27" layer="22" ratio="12" rot="MR0">v1.0 03/16/2020</text>
-<text x="43.942" y="13.081" size="1.27" layer="22" ratio="12" rot="MR0">by Seeed Studio</text>
+<text x="43.942" y="13.081" size="1.27" layer="22" ratio="12" rot="MR0">by Longan Labs</text>
 <text x="18.9865" y="9.525" size="0.889" layer="21" ratio="11">CANH</text>
 <text x="14.0335" y="9.525" size="0.889" layer="21" ratio="11">CANL</text>
@@
 <wire x1="55.245" y1="31.75" x2="55.245" y2="24.13" width="0.127" layer="22"/>
 <wire x1="55.245" y1="24.13" x2="62.23" y2="24.13" width="0.127" layer="22"/>
-<text x="43.942" y="10.414" size="1.27" layer="22" ratio="12" rot="MR0">wiki.seeed.cc/can</text>
+<text x="43.942" y="10.414" size="1.27" layer="22" ratio="12" rot="MR0">longan-labs.cc</text>
 <text x="16.383" y="40.259" size="0.8128" layer="22" ratio="12" rot="MR270">CAN OPEN</text>
 <text x="24.003" y="39.878" size="1.016" layer="22" ratio="12" rot="MR270">OBD-II</text>
@@
 <attribute name="VALUE" x="6.35" y="1.9685" size="0.8128" layer="27" ratio="10"/>
 </element>
-<element name="U$1" library="Logo" package="LOGO_SILK" value="" x="32.893" y="24.13" smashed="yes" rot="MR0"/>
 <element name="J1" library="Connector" package="DB9-MEAL" value="" x="9.525" y="31.877" smashed="yes" rot="R270">
 <attribute name="NAME" x="7.5235" y="30.1155" size="0.889" layer="37" ratio="11"/>
@@
 <attribute name="VALUE" x="19.558" y="15.748" size="0.635" layer="27" ratio="10" align="center"/>
 </element>
+<element name="U$1" library="Longan-LOGO" package="LONGAN-SILK-SMALLER" value="" x="45.212" y="18.923" rot="MR0"/>
 </elements>
 <signals>
